Commit message: more accurate ro hand tip

File: robots/hands/ro_hand/ro_hand_left.urdf (robot description, URDF)
Before this commit: robot rohand_left, 31 links, 30 joints
Joints:
- joint if_tip_joint: origin xyz=-0.048 -0.005 -0.014 rpy=0 0 0 -> xyz=-0.047 -0.004 -0.013 rpy=0 0 0
- joint lf_tip_joint: origin xyz=-0.032 -0.012 -0.014 rpy=0 0 0 -> xyz=-0.032 -0.01 -0.012 rpy=0 0 0
- joint mf_tip_joint: origin xyz=-0.048 -0.008 -0.014 rpy=0 0 0 -> xyz=-0.047 -0.007 -0.014 rpy=0 0 0

File: robots/hands/ro_hand/ro_hand_right.urdf (robot description, URDF)
Before this commit: robot rohand_right, 31 links, 30 joints
Links:
- link if_tip_link: geometry visual box size=0.003 0.003 0.003
- link lf_tip_link: geometry visual box size=0.003 0.003 0.003
- link mf_tip_link: geometry visual box size=0.003 0.003 0.003
- link rf_tip_link: geometry visual box size=0.003 0.003 0.003
- link th_tip_link: geometry visual box size=0.003 0.003 0.003
Joints:
- joint if_tip_joint: origin xyz=0 0 0 rpy=0 0 0 -> xyz=-0.046 -0.009 -0.014 rpy=0 0 0
- joint lf_tip_joint: origin xyz=0 0 0 rpy=0 0 0 -> xyz=-0.032 -0.004 -0.012 rpy=0 0 0
- joint mf_tip_joint: origin xyz=0 0 0 rpy=0 0 0 -> xyz=-0.047 -0.007 -0.014 rpy=0 0 0
- joint rf_tip_joint: origin xyz=0 0 0 rpy=0 0 0 -> xyz=-0.046 -0.003 -0.017 rpy=0 0 0
- joint th_tip_joint: origin xyz=0 0 0 rpy=0 0 0 -> xyz=-0.011 -0.023 -0.009 rpy=0 0 0

Commit message: oh urdf fix for teleop

File: robots/hands/ro_hand/ro_hand_left.urdf (robot description, URDF)
Before this commit: robot rohand_left, 31 links, 30 joints
Links:
- added link world_root
Joints:
- added joint root_transform: type fixed, parent world_root, child base_link, origin xyz=0 0 0 rpy=0 1.5707963 3.14
- joint if_connecting_link: limit (none) -> lower=-3.14 upper=3.14 effort=0 velocity=0; type continuous -> fixed
- joint if_distal_link: limit (none) -> lower=-3.14 upper=3.14 effort=0 velocity=0; type continuous -> revolute
- joint if_proximal_link: limit (none) -> lower=-1.466 upper=0.0 effort=0 velocity=0; mimic joint=if_slider_link multiplier=-75.052450 offset=-0.055446 -> (none); type continuous -> revolute
- joint if_slider_abpart_link: limit (none) -> lower=-3.14 upper=3.14 effort=0 velocity=0; type continuous -> fixed
- joint if_slider_link: type prismatic -> fixed
- joint lf_connecting_link: type continuous -> fixed
- joint lf_distal_link: limit (none) -> lower=-3.14 upper=3.14 effort=0 velocity=0; type continuous -> revolute
- joint lf_proximal_link: limit (none) -> lower=-1.455 upper=0.0 effort=0 velocity=0; mimic joint=lf_slider_link multiplier=-74.278679 offset=-0.049528 -> (none); type continuous -> revolute
- joint lf_slider_abpart_link: type continuous -> fixed
- joint lf_slider_link: type prismatic -> fixed
- joint mf_connecting_link: limit (none) -> lower=-3.14 upper=3.14 effort=0 velocity=0; type continuous -> fixed
- joint mf_distal_link: limit (none) -> lower=-3.14 upper=3.14 effort=0 velocity=0; type continuous -> revolute
- joint mf_proximal_link: limit (none) -> lower=-1.466 upper=0.00 effort=0 velocity=0; mimic joint=mf_slider_link multiplier=-74.008909 offset=-0.065644 -> (none); type continuous -> revolute
- joint mf_slider_abpart_link: type continuous -> fixed
- joint mf_slider_link: type prismatic -> fixed
- joint rf_connecting_link: type continuous -> fixed
- joint rf_distal_link: limit (none) -> lower=-3.14 upper=3.14 effort=0 velocity=0; type continuous -> revolute
- joint rf_proximal_link: limit (none) -> lower=-1.460 upper=0.0 effort=0 velocity=0; mimic joint=rf_slider_link multiplier=-74.604806 offset=-0.051526 -> (none); type continuous -> revolute
- joint rf_slider_abpart_link: type continuous -> fixed
- joint rf_slider_link: type prismatic -> fixed
- joint th_connecting_link: limit (none) -> lower=-3.14 upper=3.14 effort=0 velocity=0; type continuous -> fixed
- joint th_distal_link: limit (none) -> lower=-3.14 upper=0.0 effort=0 velocity=0; type continuous -> revolute
- joint th_proximal_link: limit (none) -> lower=-0.5 upper=0.0 effort=0 velocity=0; mimic joint=th_slider_link multiplier=-70.405870 offset=0.020045 -> (none); type continuous -> revolute
- joint th_slider_link: type prismatic -> fixed

File: robots/hands/ro_hand/ro_hand_right.urdf (robot description, URDF)
Before this commit: robot rohand_right, 31 links, 30 joints
Links:
- added link world_root
Joints:
- added joint root_transform: type fixed, parent world_root, child base_link, origin xyz=0 0 0 rpy=0 1.5707963 3.14
- joint if_connecting_link: limit (none) -> lower=-3.14 upper=3.14 effort=0 velocity=0; type continuous -> fixed
- joint if_distal_link: limit (none) -> lower=-3.14 upper=3.14 effort=0 velocity=0; type continuous -> revolute
- joint if_proximal_link: limit (none) -> lower=-1.466 upper=0.0 effort=0 velocity=0; mimic joint=if_slider_link multiplier=-75.052450 offset=-0.055446 -> (none); type continuous -> revolute
- joint if_slider_abpart_link: limit (none) -> lower=-3.14 upper=3.14 effort=0 velocity=0; type continuous -> fixed
- joint if_slider_link: type prismatic -> fixed
- joint lf_connecting_link: type continuous -> fixed
- joint lf_distal_link: limit (none) -> lower=-3.14 upper=3.14 effort=0 velocity=0; type continuous -> revolute
- joint lf_proximal_link: limit (none) -> lower=-1.455 upper=0.0 effort=0 velocity=0; mimic joint=lf_slider_link multiplier=-74.278679 offset=-0.049528 -> (none); type continuous -> revolute
- joint lf_slider_abpart_link: type continuous -> fixed
- joint lf_slider_link: type prismatic -> fixed
- joint mf_connecting_link: type continuous -> fixed
- joint mf_distal_link: limit (none) -> lower=-3.14 upper=3.14 effort=0 velocity=0; type continuous -> revolute
- joint mf_proximal_link: limit (none) -> lower=-1.466 upper=0.00 effort=0 velocity=0; mimic joint=mf_slider_link multiplier=-74.008909 offset=-0.065644 -> (none); type continuous -> revolute
- joint mf_slider_abpart_link: type continuous -> fixed
- joint mf_slider_link: type prismatic -> fixed
- joint rf_connecting_link: type continuous -> fixed
- joint rf_distal_link: limit (none) -> lower=-3.14 upper=3.14 effort=0 velocity=0; type continuous -> revolute
- joint rf_proximal_link: limit (none) -> lower=-1.460 upper=0.0 effort=0 velocity=0; mimic joint=rf_slider_link multiplier=-74.604806 offset=-0.051526 -> (none); type continuous -> revolute
- joint rf_slider_abpart_link: type continuous -> fixed
- joint rf_slider_link: type prismatic -> fixed
- joint th_connecting_link: limit (none) -> lower=-3.14 upper=3.14 effort=0 velocity=0; type continuous -> fixed
- joint th_distal_link: limit (none) -> lower=-3.14 upper=0.0 effort=0 velocity=0; type continuous -> revolute
- joint th_proximal_link: limit (none) -> lower=-0.5 upper=0.0 effort=0 velocity=0; mimic joint=th_slider_link multiplier=-70.405870 offset=0.020045 -> (none); type continuous -> revolute
- joint th_slider_link: type prismatic -> fixed
