Commit message: update omni hand

File: robots/hands/omni_hand/omni_hand_left.urdf (robot description, URDF)
Before this commit: robot O12-T2-l-URDF, 25 links, 24 joints
Links:
- removed link index_Virtual_Point
- removed link middle_Virtual_Point
- removed link pinky_Virtual_Point
- removed link ring_Virtual_Point
- removed link thumb_Virtual_Point
- added link index_distal_vertices_virtual_coordinates; collision sphere radius=0.001
- added link middle_distal_vertices_virtual_coordinates; collision sphere radius=0.001
- added link pinky_distal_vertices_virtual_coordinates; collision sphere radius=0.001
- added link ring_distal_vertices_virtual_coordinates; collision sphere radius=0.001
- added link thumb_distal_vertices_virtual_coordinates; collision sphere radius=0.001
- link hand_base_link: mass 0.114844256740337 -> 0.831592534870634; geometry collision box size=0.05 0.09 0.09; collision cylinder length=0.01 radius=0.032
- link index_distal: mass 0.00258259740989255 -> 0.00919575167024177; geometry collision cylinder length=0.02 radius=0.01; visual mesh filename=meshes/index_distal.STL
- link index_metacarpals: mass 0.00107972492721203 -> 0.00769184155607912; geometry visual mesh filename=meshes/index_metacarpals.STL
- link index_middle: mass 0.00270775197321639 -> 0.00438956668936868; geometry collision cylinder length=0.022 radius=0.01; visual mesh filename=meshes/index_middle.STL
- link index_proximal: mass 0.00477960256059446 -> 0.00942126624293676; geometry collision cylinder length=0.038 radius=0.01; visual mesh filename=meshes/index_proximal.STL
- link middle_distal: mass 0.00258260265037946 -> 0.00919573396837047; geometry collision cylinder length=0.018 radius=0.01; visual mesh filename=meshes/middle_distal.STL
- link middle_metacarpals: mass 0.00107972492722234 -> 0.00637102949978218; geometry visual mesh filename=meshes/middle_metacarpals.STL
- link middle_middle: mass 0.00314204671441198 -> 0.00495728561619528; geometry collision cylinder length=0.028 radius=0.01; visual mesh filename=meshes/middle_middle.STL
- link middle_proximal: mass 0.00551224266379775 -> 0.0105445601098368; geometry collision cylinder length=0.04 radius=0.01; visual mesh filename=meshes/middle_proximal.STL
- link pinky_distal: mass 0.0025825918864764 -> 0.00919575186910556; geometry collision cylinder length=0.018 radius=0.01; visual mesh filename=meshes/ring_distal.STL
- link pinky_middle: mass 0.00270775341133159 -> 0.0047795328266326; geometry collision cylinder length=0.028 radius=0.01; visual mesh filename=meshes/ring_middle.STL
- link pinky_proximal: mass 0 -> 0.0047795328266326; geometry collision cylinder length=0.035 radius=0.01; visual mesh filename=meshes/ring_proximal.STL
- link ring_distal: mass 0.00258259191907092 -> 0.00919575186910556; geometry collision cylinder length=0.018 radius=0.01; visual mesh filename=meshes/ring_distal.STL
- link ring_middle: mass 0.00270775337558511 -> 0.0047795328266326; geometry collision cylinder length=0.028 radius=0.01; visual mesh filename=meshes/ring_middle.STL
- link ring_proximal: mass 0.00477953283061717 -> 0.0047795328266326; geometry collision cylinder length=0.035 radius=0.01; visual mesh filename=meshes/ring_proximal.STL
- link thumb_distal: mass 0.00521800678366716 -> 0.0166245749238282; geometry collision cylinder length=0.03 radius=0.01; visual mesh filename=meshes/l_thumb_distal.STL
- link thumb_metacarpals: mass 0.017091 -> 0.0238744814807847; geometry collision box size=0.064 0.023 0.03; visual mesh filename=meshes/l_thumb_metacarpals.STL
- link thumb_metacarpals_base1: mass 0.00393646023590197 -> 0.0487218724123021; geometry visual mesh filename=meshes/l_thumb_metacarpals_base1.STL
- link thumb_metacarpals_base2: mass 0.00171679371228901 -> 0.00527730022012764; geometry collision box size=0.035 0.006 0.02; visual mesh filename=meshes/l_thumb_metacarpals_base2.STL
- link thumb_proximal: mass 0.00522967384448073 -> 0.015089750823072; geometry collision cylinder length=0.02 radius=0.01; visual mesh filename=meshes/l_thumb_proximal.STL
Joints:
- removed joint index_Virtual_Point-none
- removed joint index_dip
- removed joint index_mcp_pitch
- removed joint index_mcp_roll
- removed joint index_pip
- removed joint middle_Virtual_Point-none
- removed joint middle_dip
- removed joint middle_mcp_pitch
- removed joint middle_mcp_roll
- removed joint middle_pip
- removed joint pinky_Virtual_Point-none
- removed joint pinky_dip
- removed joint pinky_mcp_pitch
- removed joint pinky_pip
- removed joint ring_Virtual_Point-none
- removed joint ring_dip
- removed joint ring_mcp_pitch
- removed joint ring_pip
- removed joint thumb_Virtual_Point-none
- removed joint thumb_cmc_pitch
- removed joint thumb_cmc_roll
- removed joint thumb_cmc_yaw
- removed joint thumb_ip
- removed joint thumb_mcp
- added joint index_abad_joint: type revolute, parent hand_base_link, child index_metacarpals, origin xyz=-0.0134 -0.030778 0.11936 rpy=0 0 0, axis 1 0 0, limit lower=-0.26 upper=0.26 effort=1.001 velocity=2.16
- added joint index_dip_joint: type revolute, parent index_middle, child index_distal, origin xyz= 0.0058514  0 0.026478 rpy=0 0 0, axis 0 1 0, limit lower=0 upper=1.31 effort=0.216 velocity=2.85, mimic joint=index_pip_joint multiplier=1.0362 offset=0
- added joint index_mcp_joint: type revolute, parent index_metacarpals, child index_proximal, origin xyz=0.01357 0 0 rpy=0 0 0, axis 0 1 0, limit lower=0 upper=1.33 effort=0.42 velocity=2.22
- added joint index_pip_joint: type revolute, parent index_proximal, child index_middle, origin xyz=-0.0044047 0 0.039781 rpy=0 0 0, axis 0 1 0, limit lower=0 upper=1.48 effort=0.216 velocity=2.49
- added joint index_tip: type fixed, parent index_distal, child index_distal_vertices_virtual_coordinates, origin xyz=-0.01465 0 0.02533 rpy=0 0 0
- added joint middle_abad_joint: type revolute, parent hand_base_link, child middle_metacarpals, origin xyz=-0.0134 -0.0066607 0.11936 rpy=0 0 0, axis 1 0 0, limit lower=-0.26 upper=0.26 effort=1.031 velocity=2.16
- added joint middle_dip_joint: type revolute, parent middle_middle, child middle_distal, origin xyz= 0.005529  0 0.031336 rpy=0 0 0, axis 0 1 0, limit lower=0 upper=1.31 effort=0.136 velocity=2.48, mimic joint=middle_pip_joint multiplier=1.0924 offset=0
- added joint middle_mcp_joint: type revolute, parent middle_metacarpals, child middle_proximal, origin xyz=0.01337 0 0 rpy=0 0 0, axis 0 1 0, limit lower=0 upper=1.33 effort=0.413 velocity=2.22
- added joint middle_pip_joint: type revolute, parent middle_proximal, child middle_middle, origin xyz=-0.0040396 0 0.044837 rpy=0 0 0, axis 0 1 0, limit lower=0 upper=1.71 effort=0.136 velocity=2.16
- added joint middle_tip: type fixed, parent middle_distal, child middle_distal_vertices_virtual_coordinates, origin xyz=-0.01465 0 0.02533 rpy=0 0 0
- added joint pinky_dip_joint: type revolute, parent pinky_middle, child pinky_distal, origin xyz= 0.006162  0 0.026407 rpy=0 0 0, axis 0 1 0, limit lower=0 upper=1.31 effort=0.444 velocity=2.62, mimic joint=pinky_mcp_joint multiplier=0.9394 offset=0
- added joint pinky_mcp_joint: type revolute, parent hand_base_link, child pinky_proximal, origin xyz=0.0001598 0.033576 0.11272 rpy=0.0 0.0 0.0, axis 0 1 0, limit lower=0 upper=1.38 effort=0.444 velocity=2.54
- added joint pinky_pip_joint: type revolute, parent pinky_proximal, child pinky_middle, origin xyz=-0.0039371 0 0.03983 rpy=0 0 0, axis 0 1 0, limit lower=0 upper=1.57 effort=0.444 velocity=2.29, mimic joint=pinky_mcp_joint multiplier=0.877 offset=0
- added joint pinky_tip_joint: type fixed, parent pinky_distal, child pinky_distal_vertices_virtual_coordinates, origin xyz=-0.01465 0 0.02533 rpy=0 0 0
- added joint ring_dip_joint: type revolute, parent ring_middle, child ring_distal, origin xyz= 0.006162  0 0.026407 rpy=0 0 0, axis 0 1 0, limit lower=0 upper=1.31 effort=0.444 velocity=2.62, mimic joint=ring_mcp_joint multiplier=0.9394 offset=0
- added joint ring_mcp_joint: type revolute, parent hand_base_link, child ring_proximal, origin xyz=0.0001598 0.013518 0.11972 rpy=0.0 0.0 0.0, axis 0 1 0, limit lower=0 upper=1.38 effort=0.444 velocity=2.54
- added joint ring_pip_joint: type revolute, parent ring_proximal, child ring_middle, origin xyz=-0.0039371 0 0.03983 rpy=0 0 0, axis 0 1 0, limit lower=0 upper=1.57 effort=0.444 velocity=2.29, mimic joint=ring_mcp_joint multiplier=0.877 offset=0
- added joint ring_tip_joint: type fixed, parent ring_distal, child ring_distal_vertices_virtual_coordinates, origin xyz=-0.01465 0 0.02533 rpy=0 0 0
- added joint thumb_abad_joint: type revolute, parent thumb_metacarpals_base1, child thumb_metacarpals_base2, origin xyz=0.029071 0 0.0033014 rpy=0 0.95993 0, axis 0 -1 0, limit lower=0 upper=1.22 effort=0.317 velocity=2.33
- added joint thumb_dip_joint: type revolute, parent thumb_proximal, child thumb_distal, origin xyz= -0.0025791  0 0.034516 rpy=0 0 0, axis 0 -1 0, limit lower=-1.31 upper=0 effort=0.92 velocity=1.9, mimic joint=thumb_pip_joint multiplier=0.8068 offset=0
- added joint thumb_mcp_joint: type revolute, parent thumb_metacarpals_base2, child thumb_metacarpals, origin xyz=0.0016774 0.0068611 0.022935 rpy=0 0.66452 1.5708, axis 0 -1 0, limit lower=-0.85 upper=0 effort=0.8 velocity=1.35
- added joint thumb_pip_joint: type revolute, parent thumb_metacarpals, child thumb_proximal, origin xyz=0.0067768 0 0.05582 rpy=0 0 0, axis 0 -1 0, limit lower=-1.29 upper=0 effort=0.92 velocity=1.87
- added joint thumb_roll_joint: type revolute, parent hand_base_link, child thumb_metacarpals_base1, origin xyz=-0.00148 -0.022278 0.04025 rpy=2.0246 0 0, axis 1 0 0, limit lower=-0.66 upper=0 effort=0.134 velocity=2.38
- added joint thumb_tips: type fixed, parent thumb_distal, child thumb_distal_vertices_virtual_coordinates, origin xyz=-0.01107 0 0.02778 rpy=0 0 0, axis 0 0 0

File: robots/hands/omni_hand/omni_hand_right.urdf (robot description, URDF)
Before this commit: robot O12-T2-r-URDF, 25 links, 24 joints
Links:
- removed link index_Virtual_Point
- removed link middle_Virtual_Point
- removed link pinky_Virtual_Point
- removed link ring_Virtual_Point
- removed link thumb_Virtual_Point
- added link index_distal_vertices_virtual_coordinates; collision sphere radius=0.001
- added link middle_distal_vertices_virtual_coordinates; collision sphere radius=0.001
- added link pinky_distal_vertices_virtual_coordinates; collision sphere radius=0.001
- added link ring_distal_vertices_virtual_coordinates; collision sphere radius=0.001
- added link thumb_distal_vertices_virtual_coordinates; collision sphere radius=0.001
- link hand_base_link: mass 0.114811257443678 -> 0.831592534870634; geometry collision box size=0.05 0.09 0.09; collision cylinder length=0.01 radius=0.032
- link index_distal: mass 0.00258259704107596 -> 0.00919575167024177; geometry collision cylinder length=0.02 radius=0.01; visual mesh filename=meshes/index_distal.STL
- link index_metacarpals: mass 0.00107972483821526 -> 0.00769184155607912; geometry visual mesh filename=meshes/index_metacarpals.STL
- link index_middle: mass 0.00270775195657711 -> 0.00438956668936868; geometry collision cylinder length=0.022 radius=0.01; visual mesh filename=meshes/index_middle.STL
- link index_proximal: mass 0.0047795679529425 -> 0.00942126624293676; geometry collision cylinder length=0.038 radius=0.01; visual mesh filename=meshes/index_proximal.STL
- link middle_distal: mass 0.00258260294313138 -> 0.00919573396837047; geometry collision cylinder length=0.018 radius=0.01; visual mesh filename=meshes/middle_distal.STL
- link middle_metacarpals: mass 0.00107972484789827 -> 0.00637102949978218; geometry visual mesh filename=meshes/middle_metacarpals.STL
- link middle_middle: mass 0.00314204808883818 -> 0.00495728561619528; geometry collision cylinder length=0.028 radius=0.01; visual mesh filename=meshes/middle_middle.STL
- link middle_proximal: mass 0.0055122415444485 -> 0.0105445601098368; geometry collision cylinder length=0.04 radius=0.01; visual mesh filename=meshes/middle_proximal.STL
- link pinky_distal: mass 0.00258259141809727 -> 0.00919575186910556; geometry collision cylinder length=0.018 radius=0.01; visual mesh filename=meshes/ring_distal.STL
- link pinky_middle: mass 0.00270775345292578 -> 0.0047795328266326; geometry collision cylinder length=0.028 radius=0.01; visual mesh filename=meshes/ring_middle.STL
- link pinky_proximal: mass 0.00477953323340541 -> 0.0047795328266326; geometry collision cylinder length=0.035 radius=0.01; visual mesh filename=meshes/ring_proximal.STL
- link ring_distal: mass 0.00258259127175773 -> 0.00919575186910556; geometry collision cylinder length=0.018 radius=0.01; visual mesh filename=meshes/ring_distal.STL
- link ring_middle: mass 0.0027077533496335 -> 0.0047795328266326; geometry collision cylinder length=0.028 radius=0.01; visual mesh filename=meshes/ring_middle.STL
- link ring_proximal: geometry collision cylinder length=0.035 radius=0.01; visual mesh filename=meshes/ring_proximal.STL
- link thumb_distal: mass 0.00521800975168049 -> 0.0166245749238282; geometry collision cylinder length=0.03 radius=0.01; visual mesh filename=meshes/r_thumb_distal.STL
- link thumb_metacarpals: mass 0.0170904824194818 -> 0.0238744814807847; geometry collision box size=0.064 0.023 0.03; visual mesh filename=meshes/r_thumb_metacarpals.STL
- link thumb_metacarpals_base1: mass 0.00393646374828629 -> 0.0487218724123021; geometry visual mesh filename=meshes/r_thumb_metacarpals_base1.STL
- link thumb_metacarpals_base2: mass 0.00171679583795965 -> 0.00527730022012764; geometry collision box size=0.035 0.006 0.02; visual mesh filename=meshes/r_thumb_metacarpals_base2.STL
- link thumb_proximal: mass 0.00522967724458737 -> 0.015089750823072; geometry collision cylinder length=0.02 radius=0.01; visual mesh filename=meshes/r_thumb_proximal.STL
Joints:
- removed joint index_Virtual_Point-none
- removed joint index_dip
- removed joint index_mcp_pitch
- removed joint index_mcp_roll
- removed joint index_pip
- removed joint middle_Virtual_Point-none
- removed joint middle_dip
- removed joint middle_mcp_pitch
- removed joint middle_mcp_roll
- removed joint middle_pip
- removed joint pinky_Virtual_Point-none
- removed joint pinky_dip
- removed joint pinky_mcp_pitch
- removed joint pinky_pip
- removed joint ring_Virtual_Point-none
- removed joint ring_dip
- removed joint ring_mcp_pitch
- removed joint ring_pip
- removed joint thumb_Virtual_Point-none
- removed joint thumb_cmc_pitch
- removed joint thumb_cmc_roll
- removed joint thumb_cmc_yaw
- removed joint thumb_ip
- removed joint thumb_mcp
- added joint index_abad_joint: type revolute, parent hand_base_link, child index_metacarpals, origin xyz=-0.0134 0.030778 0.11936 rpy=0 0 0, axis 1 0 0, limit lower=-0.26 upper=0.26 effort=1.001 velocity=2.16
- added joint index_dip_joint: type revolute, parent index_middle, child index_distal, origin xyz= 0.0058514  0 0.026478 rpy=0 0 0, axis 0 1 0, limit lower=0 upper=1.31 effort=0.216 velocity=2.85, mimic joint=index_pip_joint multiplier=1.0362 offset=0
- added joint index_mcp_joint: type revolute, parent index_metacarpals, child index_proximal, origin xyz=0.01357 0 0 rpy=0 0 0, axis 0 1 0, limit lower=0 upper=1.33 effort=0.42 velocity=2.22
- added joint index_pip_joint: type revolute, parent index_proximal, child index_middle, origin xyz=-0.0044047 0 0.039781 rpy=0 0 0, axis 0 1 0, limit lower=0 upper=1.48 effort=0.216 velocity=2.49
- added joint index_tip: type fixed, parent index_distal, child index_distal_vertices_virtual_coordinates, origin xyz=-0.01465 0 0.02533 rpy=0 0 0
- added joint middle_abad_joint: type revolute, parent hand_base_link, child middle_metacarpals, origin xyz=-0.0134 0.0066607 0.11936 rpy=0 0 0, axis 1 0 0, limit lower=-0.26 upper=0.26 effort=1.031 velocity=2.16
- added joint middle_dip_joint: type revolute, parent middle_middle, child middle_distal, origin xyz= 0.005529  0 0.031336 rpy=0 0 0, axis 0 1 0, limit lower=0 upper=1.31 effort=0.136 velocity=2.48, mimic joint=middle_pip_joint multiplier=1.0924 offset=0
- added joint middle_mcp_joint: type revolute, parent middle_metacarpals, child middle_proximal, origin xyz=0.01337 0 0 rpy=0 0 0, axis 0 1 0, limit lower=0 upper=1.33 effort=0.413 velocity=2.22
- added joint middle_pip_joint: type revolute, parent middle_proximal, child middle_middle, origin xyz=-0.0040396 0 0.044837 rpy=0 0 0, axis 0 1 0, limit lower=0 upper=1.71 effort=0.136 velocity=2.16
- added joint middle_tip: type fixed, parent middle_distal, child middle_distal_vertices_virtual_coordinates, origin xyz=-0.01465 0 0.02533 rpy=0 0 0
- added joint pinky_dip_joint: type revolute, parent pinky_middle, child pinky_distal, origin xyz= 0.006162  0 0.026407 rpy=0 0 0, axis 0 1 0, limit lower=0 upper=1.31 effort=0.444 velocity=2.62, mimic joint=pinky_mcp_joint multiplier=0.9394 offset=0
- added joint pinky_mcp_joint: type revolute, parent hand_base_link, child pinky_proximal, origin xyz=0.0001598 -0.033576 0.11272 rpy=0.0 0.0 0.0, axis 0 1 0, limit lower=0 upper=1.38 effort=0.444 velocity=2.54
- added joint pinky_pip_joint: type revolute, parent pinky_proximal, child pinky_middle, origin xyz=-0.0039371 0 0.03983 rpy=0 0 0, axis 0 1 0, limit lower=0 upper=1.57 effort=0.444 velocity=2.29, mimic joint=pinky_mcp_joint multiplier=0.877 offset=0
- added joint pinky_tip_joint: type fixed, parent pinky_distal, child pinky_distal_vertices_virtual_coordinates, origin xyz=-0.01465 0 0.02533 rpy=0 0 0
- added joint ring_dip_joint: type revolute, parent ring_middle, child ring_distal, origin xyz= 0.006162  0 0.026407 rpy=0 0 0, axis 0 1 0, limit lower=0 upper=1.31 effort=0.444 velocity=2.62, mimic joint=ring_mcp_joint multiplier=0.9394 offset=0
- added joint ring_mcp_joint: type revolute, parent hand_base_link, child ring_proximal, origin xyz=0.0001598 -0.013518 0.11972 rpy=0.0 0.0 0.0, axis 0 1 0, limit lower=0 upper=1.38 effort=0.444 velocity=2.54
- added joint ring_pip_joint: type revolute, parent ring_proximal, child ring_middle, origin xyz=-0.0039371 0 0.03983 rpy=0 0 0, axis 0 1 0, limit lower=0 upper=1.57 effort=0.444 velocity=2.29, mimic joint=ring_mcp_joint multiplier=0.877 offset=0
- added joint ring_tip_joint: type fixed, parent ring_distal, child ring_distal_vertices_virtual_coordinates, origin xyz=-0.01465 0 0.02533 rpy=0 0 0
- added joint thumb_abad_joint: type revolute, parent thumb_metacarpals_base1, child thumb_metacarpals_base2, origin xyz=0.029071 0 0.0033014 rpy=0 0.95993 0, axis 0 -1 0, limit lower=-1.22 upper=0 effort=0.317 velocity=2.33
- added joint thumb_dip_joint: type revolute, parent thumb_proximal, child thumb_distal, origin xyz= -0.0025791  0 0.034516 rpy=0 0 0, axis 0 -1 0, limit lower=-1.31 upper=0 effort=0.92 velocity=1.9, mimic joint=thumb_pip_joint multiplier=0.8068 offset=0
- added joint thumb_mcp_joint: type revolute, parent thumb_metacarpals_base2, child thumb_metacarpals, origin xyz=0.0016774 -0.0068611 0.022935 rpy=0 0.66452 -1.5708, axis 0 -1 0, limit lower=-0.85 upper=0 effort=0.8 velocity=1.35
- added joint thumb_pip_joint: type revolute, parent thumb_metacarpals, child thumb_proximal, origin xyz=0.0067768 0 0.05582 rpy=0 0 0, axis 0 -1 0, limit lower=-1.29 upper=0 effort=0.92 velocity=1.87
- added joint thumb_roll_joint: type revolute, parent hand_base_link, child thumb_metacarpals_base1, origin xyz=-0.00148 0.022278 0.04025 rpy=-2.0246 0 0, axis 1 0 0, limit lower=0 upper=0.66 effort=0.134 velocity=2.38
- added joint thumb_tips: type fixed, parent thumb_distal, child thumb_distal_vertices_virtual_coordinates, origin xyz=-0.01107 0 0.02778 rpy=0 0 0, axis 0 0 0

Commit message: fix omni left thumb abad

File: robots/hands/omni_hand/omni_hand_left.urdf (robot description, URDF)
Before this commit: robot omnihand, 25 links, 24 joints
Joints:
- joint thumb_abad_joint: limit lower=0 upper=1.22 effort=0.317 velocity=2.33 -> lower=-1.22 upper=0 effort=0.317 velocity=2.33
