Commit message: consistent limit

File: robots/hands/omni_hand/omni_hand_right.urdf (robot description, URDF)
Before this commit: robot omnihand, 25 links, 24 joints
Joints:
- joint thumb_roll_joint: axis 1 0 0 -> -1 0 0; limit lower=0 upper=0.66 effort=0.134 velocity=2.38 -> lower=-0.66 upper=0 effort=0.134 velocity=2.38
